File: first/first.kicad_pcb (KiCad board)
At the start: 2 copper layers, 287.1 x 87.5 mm, 110 parts, among them U1 Nice_Nano_V2, U2 Nice_Nano_V2

Commit message: feat:initial firmware
Other:
- board text added: "ISEN"
- board text added: "Waranty void if used for Java"
Changed lines of the file:
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@@
 		(layer "F.Fab")
 	)
+	(gr_text "Waranty void if used for Java"
+		(at 10.25 -111.75 0)
+		(layer "B.SilkS")
+		(effects
+			(font
+				(size 6 6)
+				(thickness 0.8)
+			)
+			(justify right bottom mirror)
+		)
+	)
+	(gr_text "ISEN"
+		(at 159.5 -144.25 0)
+		(layer "B.SilkS")
+		(effects
+			(font
+				(size 3 3)
+				(thickness 0.5)
+				(bold yes)
+			)
+			(justify left bottom)
+		)
+	)
 	(segment
 		(start 24.8325 -141.93)
@@
 		(polygon
 			(pts
-				(xy -6.36125 -172.68) (xy 314.13875 -173.18) (xy 319.88875 -32.43) (xy -5.36125 -32.93) (xy -6.11125 -172.68)
+				(xy -2.5 -166.5) (xy 308.75 -167.25) (xy 309.25 -54.75) (xy -2.25 -56.5)
 			)
 		)
